Commit message: controller is added

File: MYROBOT_description/urdf/mybot.xacro (robot description, xacro)
@@ -7,4 +7,10 @@
   <xacro:include filename="$(find mybot_description)/urdf/materials.xacro" />
   <xacro:include filename="$(find mybot_description)/urdf/macros.xacro" /> -->
+  <gazebo>
+  <plugin name="gazebo_ros_control" filename="libgazebo_ros_control.so">
+    <robotNamespace>/myrobot</robotNamespace>
+    <robotSimType>gazebo_ros_control/DefaultRobotHWSim</robotSimType>
+  </plugin>
+</gazebo>
 <link name="world"/>
   <joint name="fixed" type="fixed">
@@ -96,3 +102,24 @@
     <material>Gazebo/Orange</material>
   </gazebo>
+<!-- transmission -->
+<transmission name="tran1">
+    <type>transmission_interface/SimpleTransmission</type>
+    <joint name="joint1">
+      <hardwareInterface>EffortJointInterface</hardwareInterface>
+    </joint>
+    <actuator name="motor1">
+      <hardwareInterface>EffortJointInterface</hardwareInterface>
+      <mechanicalReduction>1</mechanicalReduction>
+    </actuator>
+  </transmission>
+  <transmission name="tran2">
+    <type>transmission_interface/SimpleTransmission</type>
+    <joint name="joint2">
+      <hardwareInterface>EffortJointInterface</hardwareInterface>
+    </joint>
+    <actuator name="motor2">
+      <hardwareInterface>EffortJointInterface</hardwareInterface>
+      <mechanicalReduction>1</mechanicalReduction>
+    </actuator>
+  </transmission>
 </robot>

Commit message: beginner tutorials added

File: MYROBOT_description/urdf/mybot.xacro (robot description, xacro)
@@ -3,14 +3,21 @@
   <xacro:property name="cameraSize" value="0.05"/>
   <xacro:property name="cameraMass" value="0.1"/>
+  <xacro:property name="mass" value="1"/>
+  <xacro:property name="width" value="0.1" /> <!-- Link 1 -->
+   <xacro:property name="height1" value="1" /> <!-- Link 1 -->
+  <xacro:property name="height2" value="0.5" /> <!-- Link 2 -->
+  <xacro:property name="height3" value="0.3" /> <!-- Link 3 -->
+  <xacro:property name="camera_link" value="0.05" /> <!-- Size of square 'camera' box -->
+  <xacro:property name="axel_offset" value="0.05" /> <!-- Space btw top of beam and the each joint -->
   <xacro:property name="link1_length" value="1.5"/>
-  <!-- <xacro:include filename="$(find mybot_description)/urdf/mybot.gazebo" />
-  <xacro:include filename="$(find mybot_description)/urdf/materials.xacro" />
+  <xacro:include filename="$(find MYROBOT_description)/urdf/mybot.gazebo" />
+  <!--<xacro:include filename="$(find mybot_description)/urdf/materials.xacro" />
   <xacro:include filename="$(find mybot_description)/urdf/macros.xacro" /> -->
-  <gazebo>
+  <!--<gazebo>
   <plugin name="gazebo_ros_control" filename="libgazebo_ros_control.so">
     <robotNamespace>/myrobot</robotNamespace>
     <robotSimType>gazebo_ros_control/DefaultRobotHWSim</robotSimType>
   </plugin>
-</gazebo>
+</gazebo> -->
 <link name="world"/>
   <joint name="fixed" type="fixed">
@@ -18,25 +25,26 @@
     <child link="link1"/>
   </joint>
-  <!-- Base Link -->
+ <!-- Base Link -->
   <link name="link1">
     <collision>
-      <origin rpy="0 0 0" xyz="0 0 1.0"/>
+      <origin xyz="0 0 ${height1/2}" rpy="0 0 0"/>
       <geometry>
-        <box size="0.1 0.1 2"/>
+  <box size="${width} ${width} ${height1}"/>
       </geometry>
     </collision>
     <visual>
-      <origin rpy="0 0 0" xyz="0 0 1.0"/>
+      <origin xyz="0 0 ${height1/2}" rpy="0 0 0"/>
       <geometry>
-        <box size="0.1 0.1 ${link1_length}"/>
+  <box size="${width} ${width} ${height1}"/>
       </geometry>
-     <material name="blue">
-        <color rgba="0 0 .8 1"/>
-      </material>
+      <material name="orange"/>
     </visual>
     <inertial>
-      <origin rpy="0 0 0" xyz="0 0 1.0"/>
-      <mass value="1"/>
-      <inertia ixx="1.0" ixy="0.0" ixz="0.0" iyy="1.0" iyz="0.0" izz="1.0"/>
+      <origin xyz="0 0 ${height1/2}" rpy="0 0 0"/>
+      <mass value="${mass}"/>
+      <inertia
+    ixx="${mass / 12.0 * (width*width + height1*height1)}" ixy="0.0" ixz="0.0"
+    iyy="${mass / 12.0 * (height1*height1 + width*width)}" iyz="0.0"
+    izz="${mass / 12.0 * (width*width + width*width)}"/>
     </inertial>
   </link>
@@ -44,5 +52,5 @@
     <parent link="link1"/>
     <child link="link2"/>
-    <origin rpy="0 0 0" xyz="0 0.1 1.0"/>
+    <origin xyz="0 ${width} ${height1 - axel_offset}" rpy="0 0 0"/>
     <axis xyz="0 1 0"/>
     <dynamics damping="0.7"/>
@@ -51,20 +59,23 @@
   <link name="link2">
     <collision>
-      <origin rpy="0 0 0" xyz="0 0 0.45"/>
+      <origin xyz="0 0 ${height2/2 - axel_offset}" rpy="0 0 0"/>
       <geometry>
-        <box size="0.1 0.1 1"/>
+  <box size="${width} ${width} ${height2}"/>
       </geometry>
     </collision>
     <visual>
-      <origin rpy="0 1.57 0" xyz="0.2 0 0"/>
+      <origin xyz="0 0 ${height2/2 - axel_offset}" rpy="0 0 0"/>
       <geometry>
-        <box size="0.1 0.1 1"/>
+  <box size="${width} ${width} ${height2}"/>
       </geometry>
       <material name="black"/>
     </visual>
     <inertial>
-      <origin rpy="0 0 0" xyz="0.2 0.0 0.0"/>
-      <mass value="1"/>
-      <inertia ixx="1.0" ixy="0.0" ixz="0.0" iyy="1.0" iyz="0.0" izz="1.0"/>
+      <origin xyz="0 0 ${height2/2 - axel_offset}" rpy="0 0 0"/>
+      <mass value="${mass}"/>
+      <inertia
+    ixx="${mass / 12.0 * (width*width + height2*height2)}" ixy="0.0" ixz="0.0"
+    iyy="${mass / 12.0 * (height2*height2 + width*width)}" iyz="0.0"
+    izz="${mass / 12.0 * (width*width + width*width)}"/>
     </inertial>
   </link>
@@ -72,5 +83,5 @@
     <parent link="link2"/>
     <child link="link3"/>
-    <origin rpy="0 0 0" xyz="0 0.1 0.9"/>
+    <origin xyz="0 ${width} ${height2 - axel_offset*2}" rpy="0 0 0"/>
     <axis xyz="0 1 0"/>
     <dynamics damping="0.7"/>
@@ -79,27 +90,89 @@
   <link name="link3">
     <collision>
-      <origin rpy="0 0 0" xyz="0 0 0.45"/>
+      <origin xyz="0 0 ${height3/2 - axel_offset}" rpy="0 0 0"/>
       <geometry>
-        <box size="0.1 0.1 1"/>
+  <box size="${width} ${width} ${height3}"/>
       </geometry>
     </collision>
     <visual>
-      <origin rpy="0 0 0" xyz="0 0 0.45"/>
+      <origin xyz="0 0 ${height3/2 - axel_offset}" rpy="0 0 0"/>
       <geometry>
-        <!-- <box size="0.1 0.1 1"/> -->
-       <mesh filename="package://MYROBOT_description/meshes/upper_arm.dae"/>
+  <box size="${width} ${width} ${height3}"/>
       </geometry>
       <material name="orange"/>
     </visual>
     <inertial>
-      <origin rpy="0 0 0" xyz="0 0 0.45"/>
-      <mass value="1"/>
-      <inertia ixx="1.0" ixy="0.0" ixz="0.0" iyy="1.0" iyz="0.0" izz="1.0"/>
+      <origin xyz="0 0 ${height3/2 - axel_offset}" rpy="0 0 0"/>
+      <mass value="${mass}"/>
+      <inertia
+    ixx="${mass / 12.0 * (width*width + height3*height3)}" ixy="0.0" ixz="0.0"
+    iyy="${mass / 12.0 * (height3*height3 + width*width)}" iyz="0.0"
+    izz="${mass / 12.0 * (width*width + width*width)}"/>
+    </inertial>
+  </link>
+  <!-- Camera -->
+  <joint name="camera_joint" type="fixed">
+    <axis xyz="0 1 0" />
+    <origin xyz="${camera_link} 0 ${height3 - axel_offset*2}" rpy="0 0 0"/>
+    <parent link="link3"/>
+    <child link="camera_link"/>
+  </joint>
+  <!-- Camera -->
+  <link name="camera_link">
+    <collision>
+      <origin xyz="0 0 0" rpy="0 0 0"/>
+      <geometry>
+    <box size="${camera_link} ${camera_link} ${camera_link}"/>
+      </geometry>
+    </collision>
+    <visual>
+      <origin xyz="0 0 0" rpy="0 0 0"/>
+      <geometry>
+    <box size="${camera_link} ${camera_link} ${camera_link}"/>
+      </geometry>
+      <material name="red"/>
+    </visual>
+    <inertial>
+      <mass value="1e-5" />
+      <origin xyz="0 0 0" rpy="0 0 0"/>
+      <inertia ixx="1e-6" ixy="0" ixz="0" iyy="1e-6" iyz="0" izz="1e-6" />
+    </inertial>
+  </link>
+ <!-- Hokuyo Laser -->
+<joint name="hokuyo_joint" type="fixed">
+    <axis xyz="0 1 0" />
+    <origin xyz="0 0 ${height3 - axel_offset/2}" rpy="0 0 0"/>
+    <parent link="link3"/>
+    <child link="hokuyo_link"/>
+  </joint>
+  <link name="hokuyo_link">
+    <collision>
+      <origin xyz="0 0 0" rpy="0 0 0"/>
+      <geometry>
+  <box size="0.1 0.1 0.1"/>
+      </geometry>
+    </collision>
+    <visual>
+      <origin xyz="0 0 0" rpy="0 0 0"/>
+      <geometry>
+        <mesh filename="package://MYROBOT_description/meshes/hokuyo.dae"/>
+      </geometry>
+    </visual>
+    <inertial>
+      <mass value="1e-5" />
+      <origin xyz="0 0 0" rpy="0 0 0"/>
+      <inertia ixx="1e-6" ixy="0" ixz="0" iyy="1e-6" iyz="0" izz="1e-6" />
     </inertial>
   </link>
  <!-- setting material of robot link -->
- <gazebo reference="link1">
+ <!--<gazebo reference="link1">
     <material>Gazebo/Orange</material>
   </gazebo>
+  <gazebo reference="link2">
+    <material>Gazebo/Blue</material>
+  </gazebo>
+  <gazebo reference="camera_link">
+    <material>Gazebo/Red</material>
+  </gazebo> -->
 <!-- transmission -->
 <transmission name="tran1">
